Commit message: map my world

File: project4/my_robot/urdf/my_robot.xacro (robot description, xacro)
@@ -190,14 +190,14 @@
   <!-- add color here -->
   <gazebo reference="chassis">
+    <material>Gazebo/Blue</material>
+  </gazebo>
+  <gazebo reference="left_wheel">
     <material>Gazebo/Red</material>
   </gazebo>
-  <gazebo reference="left_wheel">
-    <material>Gazebo/Grey</material>
-  </gazebo>
   <gazebo reference="right_wheel">
-    <material>Gazebo/Grey</material>
+    <material>Gazebo/Red</material>
   </gazebo>
   <gazebo reference="camera">
-    <material>Gazebo/White</material>
+    <material>Gazebo/white</material>
   </gazebo>
 </robot>
